File: Macroboard-v2.kicad_pcb (KiCad board)
At the start: 2 copper layers, 62.2 x 42.5 mm, 15 parts, among them Q2 Q_NPN_BEC, SW5 SW_DIP_x01, SW6 SW_DIP_x01, SW7 SW_DIP_x01, SW8 SW_DIP_x01, U1 XIAO-RP2040-DIP

Commit message: Minor changes
Other:
- board size 62.2 x 42.5 mm -> 63.6 x 42.5 mm
Changed lines of the file:
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@@
-		)
-		(fp_circle
-			(center -8.95 -10.3)
-			(end -8.95 -10.554)
-			(stroke
-				(width 0.5)
-				(type solid)
-			)
-			(fill yes)
-			(layer "F.SilkS")
 		)
 		(fp_circle
@@
 	)
 	(gr_arc
-		(start 157.38 121.27)
-		(mid 156.50132 123.39132)
-		(end 154.38 124.27)
+		(start 158.7 121.3)
+		(mid 157.82132 123.42132)
+		(end 155.7 124.3)
 		(stroke
 			(width 0.05)
@@
 	(gr_line
 		(start 98.13 81.82)
-		(end 154.38 81.82)
+		(end 155.7 81.85)
 		(stroke
 			(width 0.05)
@@
 	)
 	(gr_line
-		(start 154.38 124.27)
+		(start 155.7 124.3)
 		(end 98.13 124.27)
 		(stroke
@@
 	)
 	(gr_arc
-		(start 154.38 81.82)
-		(mid 156.50132 82.69868)
-		(end 157.38 84.82)
+		(start 155.7 81.85)
+		(mid 157.82132 82.72868)
+		(end 158.7 84.85)
 		(stroke
 			(width 0.05)
@@
 	)
 	(gr_line
-		(start 157.38 84.82)
-		(end 157.38 121.27)
+		(start 158.7 84.85)
+		(end 158.7 121.3)
 		(stroke
 			(width 0.05)
@@
 		(layer "F.CrtYd")
 	)
+	(dimension
+		(type orthogonal)
+		(layer "F.Fab")
+		(pts
+			(xy 155.6 115.7) (xy 158.7 115.6)
+		)
+		(height 13)
+		(orientation 0)
+		(format
+			(prefix "")
+			(suffix "")
+			(units 3)
+			(units_format 0)
+			(precision 4)
+			(suppress_zeroes yes)
+		)
+		(style
+			(thickness 0.1)
+			(arrow_length 1.27)
+			(text_position_mode 0)
+			(arrow_direction outward)
+			(extension_height 0.58642)
+			(extension_offset 0.5)
+			(keep_text_aligned yes)
+		)
+		(gr_text "3.1"
+			(at 157.15 127.55 0)
+			(layer "F.Fab")
+			(effects
+				(font
+					(size 1 1)
+					(thickness 0.15)
+				)
+			)
+		)
+	)
 	(via
